File: Main_Camera_Board7_with_holes.brd (EAGLE design)
At the start: 127 x 50.8 mm, 8 parts

Commit message: Added Instructions for Holes
Parts:
- moved SV1 3.57 mm to (93.5, 6.60)
Routing:
- net PWM: track 103.3 -> 100.4 mm
Other:
- board size 127 x 50.8 mm -> 126.7 x 44.2 mm
- board text added: "(0.2, 0.7 from the bottom)"
- board text added: "(0.20 from the edge, 0.7 from the top)"
- board text added: "(0.44, 0.12)"
- board text added: "(0.74,0.12)"
- board text added: "(lasers 0.875, diameter 0.3)"
- board text added: "(same as bottom,0.53 from top)"
- board text added: "5 in x 1.74 in"
- board text added: "coincident with lasers"
- board text added: "hole diameter: 0.09"
- board text removed: "5 in x 2 in"
Changed lines of the file:
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@@
 <setting verticaltext="up"/>
 </settings>
-<grid distance="0.01" unitdist="inch" unit="inch" style="lines" multiple="1" display="yes" altdistance="0.025" altunitdist="inch" altunit="inch"/>
+<grid distance="0.05" unitdist="inch" unit="inch" style="lines" multiple="1" display="yes" altdistance="0.025" altunitdist="inch" altunit="inch"/>
 <layers>
 <layer number="1" name="Top" color="4" fill="1" visible="yes" active="yes"/>
@@
 <board>
 <plain>
-<wire x1="-3.81" y1="50.8" x2="123.19" y2="50.8" width="0.4064" layer="20"/>
-<wire x1="123.19" y1="50.8" x2="123.19" y2="0" width="0.4064" layer="20"/>
-<wire x1="123.19" y1="0" x2="-3.81" y2="0" width="0.4064" layer="20"/>
-<wire x1="-3.81" y1="0" x2="-3.81" y2="50.8" width="0.4064" layer="20"/>
-<text x="-5.08" y="53.34" size="1.778" layer="51">5 in x 2 in</text>
+<wire x1="-3.81" y1="48.768" x2="122.936" y2="48.768" width="0.4064" layer="20"/>
+<wire x1="122.936" y1="48.768" x2="122.428" y2="4.572" width="0.4064" layer="20"/>
+<wire x1="122.428" y1="4.572" x2="-3.81" y2="4.572" width="0.4064" layer="20"/>
+<wire x1="-3.81" y1="4.572" x2="-3.81" y2="48.768" width="0.4064" layer="20"/>
+<text x="-3.556" y="50.292" size="1.778" layer="51">5 in x 1.74 in</text>
 <hole x="12.7" y="25.4" drill="2.2"/>
 <hole x="114.3" y="25.4" drill="2.2"/>
-<text x="91.694" y="5.08" size="1.778" layer="25" rot="R90">PWM</text>
-<text x="93.98" y="5.08" size="1.778" layer="25" rot="R90">+5V</text>
-<text x="96.774" y="5.08" size="1.778" layer="25" rot="R90">GND</text>
+<text x="91.186" y="8.382" size="1.778" layer="25" rot="R90">PWM</text>
+<text x="93.472" y="8.382" size="1.778" layer="25" rot="R90">+5V</text>
+<text x="95.758" y="8.382" size="1.778" layer="25" rot="R90">GND</text>
 <text x="-4.064" y="16.256" size="1.778" layer="25" rot="R90">GND</text>
 <text x="5.588" y="10.922" size="1.778" layer="25">PWM</text>
@@
 <text x="83.566" y="25.654" size="1.778" layer="25">LASERVOLTAGE</text>
 <hole x="58.42" y="26.543" drill="21.59"/>
+<text x="24.13" y="-3.81" size="1.778" layer="1">hole diameter: 0.09</text>
+<text x="11.43" y="7.62" size="0.762" layer="16" rot="MR0">(0.44, 0.12)</text>
+<text x="15.24" y="7.62" size="0.762" layer="16" rot="MR0">(0.74,0.12)</text>
+<text x="34.29" y="38.1" size="1.778" layer="16" rot="MR0">(same as bottom,0.53 from top)</text>
+<text x="114.3" y="31.75" size="1.778" layer="16" rot="MR0">(0.20 from the edge, 0.7 from the top)</text>
+<text x="114.3" y="26.67" size="1.778" layer="16" rot="MR0">(0.2, 0.7 from the bottom)</text>
+<text x="12.7" y="25.4" size="1.778" layer="16" rot="MR0">(lasers 0.875, diameter 0.3)</text>
+<text x="11.43" y="22.86" size="1.778" layer="16" rot="MR0">coincident with lasers</text>
+<text x="12.7" y="25.4" size="0.762" layer="16" rot="MR0">(lasers 0.875, diameter 0.3)</text>
+<text x="114.3" y="22.86" size="1.778" layer="16" rot="MR0">(lasers 0.875, diameter 0.3)</text>
+<text x="114.3" y="20.32" size="1.778" layer="16" rot="MR0">coincident with lasers</text>
 </plain>
 <attributes>
@@
 <element name="JP1" library="pinhead" package="1X02" value="" x="18.796" y="25.146" rot="R90"/>
 <element name="JP2" library="pinhead" package="1X02" value="" x="104.986" y="25.338" rot="R90"/>
-<element name="SV1" library="con-lstb" package="MA03-1" value="" x="93.218" y="3.048" rot="R180">
-<attribute name="MF" value="" x="93.218" y="3.048" size="1.778" layer="27" rot="R180" display="off"/>
-<attribute name="OC_FARNELL" value="unknown" x="93.218" y="3.048" size="1.778" layer="27" rot="R180" display="off"/>
-<attribute name="MPN" value="" x="93.218" y="3.048" size="1.778" layer="27" rot="R180" display="off"/>
-<attribute name="OC_NEWARK" value="unknown" x="93.218" y="3.048" size="1.778" layer="27" rot="R180" display="off"/>
+<element name="SV1" library="con-lstb" package="MA03-1" value="" x="93.472" y="6.604" rot="R180">
+<attribute name="MF" value="" x="93.472" y="6.604" size="1.778" layer="27" rot="R180" display="off"/>
+<attribute name="OC_FARNELL" value="unknown" x="93.472" y="6.604" size="1.778" layer="27" rot="R180" display="off"/>
+<attribute name="MPN" value="" x="93.472" y="6.604" size="1.778" layer="27" rot="R180" display="off"/>
+<attribute name="OC_NEWARK" value="unknown" x="93.472" y="6.604" size="1.778" layer="27" rot="R180" display="off"/>
 </element>
 </elements>
@@
 <signal name="GND">
 <polygon width="0.4064" layer="1">
-<vertex x="-3.81" y="50.8"/>
-<vertex x="123.19" y="50.8"/>
-<vertex x="123.19" y="0"/>
-<vertex x="-3.81" y="0"/>
+<vertex x="-3.81" y="48.768"/>
+<vertex x="122.936" y="48.768"/>
+<vertex x="122.428" y="4.572"/>
+<vertex x="-3.81" y="4.572"/>
 </polygon>
 <contactref element="U$1" pad="P$4"/>
@@
 <signal name="+5V">
 <polygon width="0.4064" layer="16">
-<vertex x="-3.81" y="0"/>
-<vertex x="123.19" y="0"/>
-<vertex x="123.19" y="50.8"/>
-<vertex x="-3.81" y="50.8"/>
+<vertex x="-3.81" y="4.572"/>
+<vertex x="122.428" y="4.572"/>
+<vertex x="122.936" y="48.768"/>
+<vertex x="-3.81" y="48.768"/>
 </polygon>
 <contactref element="U$1" pad="P$1"/>
@@
 <contactref element="SV1" pad="3"/>
 <contactref element="U$5" pad="P$5"/>
-<wire x1="90.678" y1="3.048" x2="0.254" y2="3.048" width="0.4064" layer="16"/>
-<wire x1="0.254" y1="3.048" x2="-1.778" y2="5.08" width="0.4064" layer="16"/>
 <wire x1="1.75" y1="12" x2="-0.954" y2="12" width="0.4064" layer="16"/>
 <wire x1="-0.954" y1="12" x2="-1.778" y2="11.176" width="0.4064" layer="16"/>
-<wire x1="-1.778" y1="11.176" x2="-1.778" y2="5.08" width="0.4064" layer="16"/>
+<wire x1="90.932" y1="6.604" x2="-0.508" y2="6.604" width="0.4064" layer="16"/>
+<wire x1="-0.508" y1="6.604" x2="-1.778" y2="7.874" width="0.4064" layer="16"/>
+<wire x1="-1.778" y1="7.874" x2="-1.778" y2="11.176" width="0.4064" layer="16"/>
 </signal>
 <signal name="LIGHT">
