File: Main_Camera_Board7.brd (EAGLE design)
At the start: 127 x 50.8 mm, 8 parts

Commit message: Revert "Added Instructions for Holes"
This reverts commit acebc77281901a6f31d99e6ed7f09fe10f3c712a.
Parts:
- moved JP1 2.54 mm to (16.3, 25.1)
Routing:
- net LASER: track 118.1 -> 108.4 mm
Changed lines of the file:
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@@
 <?xml version="1.0" encoding="utf-8"?>
 <!DOCTYPE eagle SYSTEM "eagle.dtd">
-<eagle version="7.6.0">
+<eagle version="7.7.0">
 <drawing>
 <settings>
@@
 <wire x1="123.19" y1="0" x2="-3.81" y2="0" width="0.4064" layer="20"/>
 <wire x1="-3.81" y1="0" x2="-3.81" y2="50.8" width="0.4064" layer="20"/>
+<wire x1="12.954" y1="22.606" x2="12.954" y2="27.686" width="0.4064" layer="51"/>
+<wire x1="109.22" y1="28.194" x2="109.22" y2="23.114" width="0.4064" layer="51"/>
 <text x="-5.08" y="53.34" size="1.778" layer="51">5 in x 2 in</text>
-<hole x="12.7" y="25.4" drill="2.2"/>
-<hole x="114.3" y="25.4" drill="2.2"/>
+<hole x="10.16" y="25.4" drill="2.2"/>
+<hole x="111.76" y="25.4" drill="2.2"/>
 <text x="91.694" y="5.08" size="1.778" layer="25" rot="R90">PWM</text>
 <text x="93.98" y="5.08" size="1.778" layer="25" rot="R90">+5V</text>
@@
 <text x="96.012" y="23.114" size="1.778" layer="25">GND</text>
 <text x="83.566" y="25.654" size="1.778" layer="25">LASERVOLTAGE</text>
-<hole x="58.42" y="26.543" drill="21.59"/>
 </plain>
 <attributes>
@@
 <element name="U$4" library="camera" package="T2I" value="T21" x="1.75" y="44.45" rot="R270"/>
 <element name="U$5" library="camera" package="T2I" value="T21" x="1.75" y="25.4" rot="R270"/>
-<element name="JP1" library="pinhead" package="1X02" value="" x="18.796" y="25.146" rot="R90"/>
+<element name="JP1" library="pinhead" package="1X02" value="" x="16.256" y="25.146" rot="R90"/>
 <element name="JP2" library="pinhead" package="1X02" value="" x="104.986" y="25.338" rot="R90"/>
 <element name="SV1" library="con-lstb" package="MA03-1" value="" x="93.218" y="3.048" rot="R180">
@@
 <wire x1="1.75" y1="33.05" x2="13.686" y2="33.05" width="1.016" layer="16"/>
 <wire x1="13.686" y1="33.05" x2="16.256" y2="30.48" width="1.016" layer="16"/>
-<wire x1="16.256" y1="30.48" x2="18.796" y2="26.416" width="1.016" layer="16"/>
+<wire x1="16.256" y1="30.48" x2="16.256" y2="26.416" width="1.016" layer="16"/>
+<wire x1="16.256" y1="26.416" x2="104.794" y2="26.416" width="1.016" layer="1"/>
 <wire x1="104.794" y1="26.416" x2="104.986" y2="26.608" width="1.016" layer="1"/>
-<wire x1="18.796" y1="26.416" x2="39.37" y2="26.416" width="0.8128" layer="1"/>
-<wire x1="39.37" y1="26.416" x2="53.086" y2="40.132" width="0.8128" layer="1"/>
-<wire x1="53.086" y1="40.132" x2="64.008" y2="40.132" width="0.8128" layer="1"/>
-<wire x1="64.008" y1="40.132" x2="77.47" y2="26.67" width="0.8128" layer="1"/>
-<wire x1="77.47" y1="26.67" x2="104.924" y2="26.67" width="0.8128" layer="1"/>
-<wire x1="104.924" y1="26.67" x2="104.986" y2="26.608" width="0.8128" layer="1"/>
 </signal>
 <signal name="N$7">
